File: PCB/Blare.pcb.kicad_pcb (KiCad board)
At the start: 2 copper layers, 97.5 x 47.5 mm, 11 parts, among them J1 Conn_01x08_Pin, SW1 SW_Push, SW2 SW_Push, SW3 SW_Push, SW4 SW_Push, U1 XIAO-ESP32-C3-SMD

Commit message: pcb and case
Parts:
- added ?: LOGO, Rocket_solder2:maskcopper-HC, F.Cu at (150.0, 88.0)
- added ?: LOGO, Rocket_solder5:maskcopper-HC, F.Cu at (150.0, 88.0)
- added ?: LOGO, Rocket_solder2:copper-HC, F.Cu at (150.0, 88.0)
Routing:
- net /SCL: track 33.0 -> 17.3 mm, vias 0 -> 2
- net Net-(U1-D1): track 36.3 -> 34.9 mm, vias 0 -> 2

Commit message: design to pcb
Parts:
- added ?: LOGO, PCB:github, F.Cu at (165.0, 79.0)
- added ?: LOGO, PCB:hive, F.Cu at (206.0, 81.0)
- added ?: LOGO, PCB:scary be, F.Cu at (150.0, 95.0)
- added ?: LOGO, Rocket_solder:stardancefinal, F.Cu at (183.0, 117.0)
- added ?: LOGO, PCB:idk2, F.Cu at (151.0, 104.0)
- added ?: LOGO, PCB:big cute bee, F.Cu at (235.0, 90.0)
- added G***: LOGO, PCB:hiveLEF, F.Cu at (237.0, 103.0)
- added G***: LOGO, PCB:moggerr, F.Cu at (176.0, 78.0)
- added G***: LOGO, PCB:bee, F.Cu at (210.0, 86.0)
Other:
- board text added: "yumm honeyyy!!"

Commit message: DRC error fixed
Parts:
- renumbered G*** to ?
Changed lines of the file:
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@@
 		(layer "F.Cu")
 		(at 237 103)
-		(property "Reference" "G***"
+		(property "Reference" ""
 			(at 0 0 0)
 			(layer "F.SilkS")
@@
 	)
 	(gr_text "BLARE\n    -by Nitish:)"
-		(at 204 80 0)
+		(at 208.164096 80.661866 0)
 		(layer "F.Cu")
 		(effects
@@
 	)
 	(gr_text "BLARE \n    -by Nitish:)"
-		(at 204 80 0)
+		(at 208.164096 80.661866 0)
 		(layer "F.Mask")
 		(effects
